File: core/core.kicad_pcb (KiCad board)
At the start: 2 copper layers, 63.5 x 63.5 mm, 78 parts, among them J1 Micro_SD_Card, J1001 CAS_stacking, J2 UART_DEBUG, J3 Conn_ARM_JTAG_SWD_10, J4 Conn_01x02, J5 USB_OTG, SW1 SW_Push, SW2 SW_Push, U1 SC18IS600, U1101 STM32F401RETx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

Commit message: Done layout
Routing:
- net /SPI2_nSS1: track 7.75 -> 63.8 mm, vias 1 -> 4
- net /I2C1_SCL: track 3.84 -> 52.1 mm, vias 0 -> 5
- net /SPI3_MOSI: track 39.5 -> 84.2 mm, vias 2 -> 3
- net /I2C1_SDA: track 5.81 -> 50.4 mm, vias 0 -> 4
- net /SPI2_nSS2: track 0.00 -> 41.8 mm, vias 0 -> 3
- net /INT6: track 19.1 -> 58.3 mm, vias 0 -> 4
- net /INT5: track 21.6 -> 54.1 mm, vias 0 -> 4
- net /SPI3_MISO: track 43.8 -> 75.7 mm, vias 3 -> 4
- net /SPI3_nSS1: track 24.5 -> 56.1 mm, vias 1 -> 3
- net /INT4: track 22.5 -> 51.6 mm, vias 0 -> 2
- net /SPI2_nSS8: track 30.5 -> 58.8 mm, vias 1 -> 2
- net /SPI3_SCK: track 53.1 -> 81.0 mm, vias 3 -> 4
- net /SPI2_nSS7: track 28.0 -> 55.8 mm, vias 1 -> 2
- net /INT3: track 22.9 -> 49.4 mm, vias 0 -> 2
- net /SPI2_nSS6: track 26.4 -> 52.7 mm, vias 1 -> 2
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
Commit message: Address comments
Connections:
- J4 pad 1: GND -> +BATT
- J4 pad 2: +BATT -> GND
- U1201 pad 19: /I2C3_SDA -> /I2C3_SCL
Routing:
- net GND: track 120.8 -> 230.6 mm, vias 10 -> 59
- net +5V: track 95.2 -> 121.9 mm
- net /SPIHS_MOSI: track 45.6 -> 66.4 mm, vias 5 -> 1
- net /I2C3_SCL: track 59.9 -> 75.3 mm, vias 3 -> 5
- net Net-(D4-Pad1): track 14.8 -> 27.2 mm
- net /SPIHS_SCK: track 61.6 -> 54.2 mm, vias 1 -> 5
- net /USER_BUTTON: track 18.1 -> 23.2 mm
- net +BATT: track 72.2 -> 67.2 mm
- net /I2C3_SDA: track 74.0 -> 70.8 mm, vias 4 -> 5
- net /UART_TX: track 24.3 -> 27.1 mm
- net /USER_LED: track 27.8 -> 30.3 mm
- net +3V3: track 350.2 -> 352.3 mm, vias 4 -> 7
- net /USB_DP: track 61.3 -> 63.0 mm
- net /USB_DM: track 64.7 -> 66.2 mm
- net /INT6: track 58.3 -> 57.1 mm
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