File: core/core.kicad_pcb (KiCad board)
At the start: 2 copper layers, 63.5 x 63.5 mm, 78 parts, among them J1 Micro_SD_Card, J1001 CAS_stacking, J2 UART_DEBUG, J3 Conn_ARM_JTAG_SWD_10, J4 Conn_01x02, J5 USB_OTG, SW1 SW_Push, SW2 SW_Push, U1 SC18IS600, U1101 STM32F401RETx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

Commit message: update layout
Parts:
- removed TP1, TP10, TP11, TP5, TP7: TestPoint, TestPoint:TestPoint_Keystone_5010-5014_Multipurpose
- J2: footprint star-common-lib:TSM-103-01-L-SV -> Connector_PinHeader_2.54mm:PinHeader_1x03_P2.54mm_Vertical
- SW1, SW2: footprint Button_Switch_SMD:SW_SPST_CK_RS282G05A3 -> Button_Switch_SMD:SW_SPST_PTS810
- moved TP6 76.3 mm to (61.5, 104.3)
- moved TP4 68.2 mm to (58.3, 65.5)
- moved TP12 54.4 mm to (73.9, 103.9)
- moved TP2 52.4 mm to (71.8, 58.3)
- moved TP3 52.4 mm to (75.8, 58.3)
- moved TP8 52.4 mm to (67.7, 58.3)
- moved C1202 50.6 mm to (185.2, 95.2), turned to 90 degrees
- moved U1 42.0 mm to (97.5, 69.1), turned to 90 degrees
- moved R1201 41.5 mm to (173.5, 101.3)
- moved C1204 41.4 mm to (173.5, 95.2)
- moved C1201 40.6 mm to (168.6, 121.7)
- moved J4 39.9 mm to (136.4, 96.3)
- moved NT1301 38.7 mm to (166.1, 92.5)
- moved C1203 38.4 mm to (168.4, 116.8), turned to 180 degrees
- moved C8 37.6 mm to (103.1, 68.6), turned to 270 degrees
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Routing:
- net +3V3: track 349.6 -> 82.3 mm, vias 7 -> 28
- net GND: track 230.6 -> 121.5 mm, vias 56 -> 43
- net /I2C3_SCL: track 75.3 -> 3.73 mm, vias 5 -> 1
- net /I2C3_SDA: track 70.8 -> 5.27 mm, vias 5 -> 1
- net /nRESET: track 104.4 -> 54.8 mm, vias 7 -> 5
- net /SPI3_SCK: track 81.8 -> 39.0 mm, vias 4 -> 2
- net /USB_VBUS: track 70.5 -> 27.7 mm, vias 3 -> 2
- net /USB_DM: track 66.2 -> 24.1 mm, vias 3 -> 2
- net /INT7: track 83.1 -> 43.4 mm, vias 4 -> 2
- net /USB_DP: track 63.0 -> 24.1 mm, vias 3 -> 2
- net /INT8: track 78.7 -> 40.9 mm, vias 4 -> 2
- net /I2C2_SDA: track 57.0 -> 20.2 mm, vias 4 -> 1
- net /I2C2_SCL: track 61.2 -> 25.1 mm, vias 4 -> 1
- net +5V: track 121.9 -> 88.1 mm, vias 2 -> 5
- net /SPI3_MOSI: track 84.2 -> 54.4 mm, vias 3 -> 2
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- added copper zone on F.Cu, net +3V3
- added copper zone on In2.Cu, net +3V3
- added copper zone on In1.Cu, net GND
- removed copper zone on B.Cu, net GND
Other:
- copper layers 2 -> 4
- net class Default: clearance 0.2 -> 0.1524
- rule trace_clearance: 0.2 -> 0.1524
- rule trace_min: 0.1778 -> 0.1524

Commit message: Second Layout pass on core
Parts:
- TP2, TP3, TP4, TP8, TP9: footprint TestPoint:TestPoint_Keystone_5010-5014_Multipurpose -> TestPoint:TestPoint_Keystone_5019_Minature; moved to B.Cu
- moved C1202 83.6 mm to (102.4, 83.8), turned to 270 degrees
- moved TP6 72.7 mm to (131.6, 85.1)
- moved C1203 72.3 mm to (104.1, 83.8), turned to 270 degrees
- moved C1201 72.0 mm to (104.9, 88.1), turned to 0 degrees
- moved TP12 70.8 mm to (140.7, 80.5)
- moved R1201 70.2 mm to (104.9, 86.4), turned to 180 degrees
- moved C1204 68.5 mm to (105.9, 83.8), turned to 270 degrees
- moved R1202 61.5 mm to (112.0, 88.1), turned to 0 degrees
- moved U1201 48.3 mm to (110.0, 84.8)
- moved C1302 41.0 mm to (122.2, 86.9)
- moved NT1301 40.5 mm to (126.2, 85.1)
- moved TP4 37.2 mm to (95.5, 67.1), turned to 270 degrees
- moved TP8 36.9 mm to (104.1, 52.8), turned to 270 degrees
- moved C1301 36.2 mm to (124.0, 86.9), turned to 270 degrees
- moved TP9 36.2 mm to (92.7, 57.7)
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Routing:
- net /I2C3_SCL: track 3.73 -> 69.1 mm, vias 1 -> 3
- net /I2C3_SDA: track 5.27 -> 60.2 mm, vias 1 -> 3
- net GND: track 121.5 -> 149.7 mm, vias 43 -> 49
- net /nRESET: track 54.8 -> 81.5 mm, vias 5 -> 8
- net +3V3: track 82.3 -> 103.7 mm, vias 28 -> 34
- net +BATT: track 69.7 -> 86.4 mm, vias 0 -> 1
- net /SPI3_nSS1: track 33.0 -> 46.7 mm
- net /SPI3_SCK: track 39.0 -> 47.9 mm, vias 2 -> 3
- net /SPI3_nSS2: track 33.0 -> 39.9 mm
- net /SPI3_MOSI: track 54.4 -> 60.1 mm, vias 2 -> 3
- net Net-(C1201-Pad2): track 0.00 -> 4.50 mm
- net /SPI3_MISO: track 46.2 -> 50.3 mm, vias 2 -> 3
- net Net-(R1201-Pad1): track 0.00 -> 2.84 mm
- net Net-(NT1301-Pad1): track 0.00 -> 2.61 mm
- net +5V: track 88.1 -> 86.4 mm
Other:
- board text added: "(probably)"
- board text added: "CAS CORE"
- board text added: "X"
- board text added: "Y"
- board text added: "Z"
- board text added: "git tag: v0.0.1"

Commit message: made layout revisions
Parts:
- removed the C1202 at (102.4, 83.8)
- added C9: 100n, Capacitor_SMD:C_0603_1608Metric, F.Cu at (136.4, 64.8)
- added D6: 40V, Diode_SMD:D_0603_1608Metric, F.Cu at (141.0, 92.7)
- added D7: LED, LED_SMD:LED_0603_1608Metric, F.Cu at (118.5, 54.7)
- added R13: 1k, Resistor_SMD:R_0603_1608Metric, F.Cu at (118.5, 59.3)
- added R14: 20, Resistor_SMD:R_0603_1608Metric, F.Cu at (114.2, 59.0)
- added U4: USBLC6-2SC6, Package_TO_SOT_SMD:SOT-23-6, F.Cu at (115.2, 55.2)
- C1201: value 100nF -> 1uF
- R6: value 1k -> 20
- TP12: value TestPoint -> SCL
- TP2: value TestPoint -> MISO
- TP3: value TestPoint -> SCK
- TP4: value TestPoint -> nSS2
- TP6: value TestPoint -> SDA
- TP8: value TestPoint -> MOSI
- TP9: value TestPoint -> nSS1
- moved R5 22.6 mm to (133.1, 69.5), turned to 270 degrees
- moved D5 22.1 mm to (133.1, 66.2), turned to 90 degrees
- moved R6 14.0 mm to (116.2, 59.0), turned to 90 degrees
- moved J2 1.53 mm to (122.6, 51.1)
- moved R4 1.53 mm to (127.6, 54.9)
- moved R3 1.53 mm to (125.1, 54.9)
- moved SW2 0.78 mm to (122.1, 56.3)
- renumbered C1203 to C1202, C1204 to C1203
Connections:
- J5 pad 2: /USB_DM -> /USB_DM_I
- J5 pad 3: /USB_DP -> /USB_DP_I
- R6 pad 1: /nRESET -> /USB_DM
- R6 pad 2: +3V3 -> Net-(R6-Pad2)
Routing:
- net GND: track 149.7 -> 162.8 mm, vias 49 -> 51
- net /USB_VBUS: track 27.7 -> 40.4 mm, vias 2 -> 3
- net /USER_LED: track 9.94 -> 21.9 mm, vias 0 -> 2
- net +5V: track 86.4 -> 93.0 mm
- net +BATT: track 86.4 -> 92.1 mm
- net /USB_DM: track 24.1 -> 20.3 mm
- net /USB_DP: track 24.1 -> 20.4 mm
- net Net-(D7-Pad1): track 0.00 -> 2.96 mm
- net /USB_DP_I: track 0.00 -> 2.52 mm
- net /USB_DM_I: track 0.00 -> 2.50 mm
- net Net-(D5-Pad1): track 3.97 -> 1.73 mm
- net /INT_I2C: track 36.5 -> 34.3 mm
- net /SPI3_MISO: track 50.3 -> 52.5 mm, vias 3 -> 2
- net Net-(R6-Pad2): track 0.00 -> 1.89 mm
- net Net-(R14-Pad1): track 0.00 -> 1.89 mm
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Other:
- board text added: "GND"
- board text added: "RX"

Commit message: update silk
Parts:
- JP2: value Jumper -> RST_JUMP
- SW1: value SW_Push -> RESET
- SW2: value SW_Push -> USER
Routing:
- net Net-(U1201-Pad7): track 0.00 -> 1.73 mm, vias 0 -> 1
- net Net-(C1201-Pad2): track 4.50 -> 6.16 mm
- net Net-(U1201-Pad8): track 0.00 -> 1.56 mm, vias 0 -> 1
Other:
- board text added: "BATTERY"
- board text added: "git tag: v0.0.2"
- board text removed: "git tag: v0.0.1"

Commit message: fix silk
Other:
- board text added: "TX"
Changed lines of the file:
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@@
   (layers
     (0 F.Cu signal)
-    (1 In1.Cu power)
-    (2 In2.Cu power)
+    (1 In1.Cu power hide)
+    (2 In2.Cu power hide)
     (31 B.Cu signal)
     (32 B.Adhes user hide)
@@
       (outputformat 1)
       (mirror false)
-      (drillshape 1)
+      (drillshape 0)
       (scaleselection 1)
-      (outputdirectory ""))
+      (outputdirectory "/tmp/floof"))
   )
   (net 0 "")
@@
     (pad 2 thru_hole oval (at 0 5.5 180) (size 2.7 3.7) (drill 1.8) (layers *.Cu *.Mask)
       (net 3 +BATT))
-    (pad 1 thru_hole roundrect (at 0 0 180) (size 2.7 3.7) (drill 1.8) (layers *.Cu *.Mask) (roundrect_rratio 0.09259299999999999)
+    (pad 1 thru_hole roundrect (at 0 0 180) (size 2.7 3.7) (drill 1.8) (layers *.Cu *.Mask) (roundrect_rratio 0.09259296296296296)
       (net 1 GND))
     (model ${KISYS3DMOD}/Connector_Molex.3dshapes/Molex_Mini-Fit_Jr_5569-02A2_2x01_P4.20mm_Horizontal.wrl
@@
     (effects (font (size 1.5 1.5) (thickness 0.3)))
   )
-  (gr_text RX (at 127.635 48.895) (layer F.SilkS)
+  (gr_text TX (at 127.635 48.895) (layer F.SilkS)
     (effects (font (size 0.75 0.75) (thickness 0.15)))
   )
@@
   (segment (start 91.694 69.342) (end 91.694 67.31) (width 0.762) (layer In1.Cu) (net 4))
   (segment (start 91.694 69.85) (end 91.694 69.342) (width 0.762) (layer In1.Cu) (net 4))
-  (via (at 95.758 86.868) (size 0.8) (drill 0.4) (layers F.Cu B.Cu) (net 4))
-  (segment (start 98.806 86.868) (end 95.758 86.868) (width 0.762) (layer F.Cu) (net 4))
-  (segment (start 100.838 97.536) (end 100.838 91.948) (width 0.762) (layer F.Cu) (net 4))
-  (segment (start 102.616 99.314) (end 100.838 97.536) (width 0.762) (layer F.Cu) (net 4))
-  (segment (start 103.124 109.474) (end 102.616 108.966) (width 0.762) (layer F.Cu) (net 4))
-  (segment (start 99.314 87.376) (end 98.806 86.868) (width 0.762) (layer F.Cu) (net 4))
-  (segment (start 99.314 90.424) (end 99.314 87.376) (width 0.762) (layer F.Cu) (net 4))
-  (segment (start 104.902 109.474) (end 103.124 109.474) (width 0.762) (layer F.Cu) (net 4))
-  (segment (start 105.41 108.966) (end 104.902 109.474) (width 0.762) (layer F.Cu) (net 4))
-  (segment (start 100.838 91.948) (end 99.314 90.424) (width 0.762) (layer F.Cu) (net 4))
-  (segment (start 102.616 108.966) (end 102.616 99.314) (width 0.762) (layer F.Cu) (net 4))
-  (segment (start 105.41 107.696) (end 105.41 108.966) (width 0.762) (layer F.Cu) (net 4))
-  (segment (start 95.758 86.868) (end 94.488 85.598) (width 1.016) (layer In1.Cu) (net 4))
-  (segment (start 94.488 85.598) (end 94.488 76.708) (width 1.016) (layer In1.Cu) (net 4))
-  (segment (start 94.488 76.708) (end 91.694 73.914) (width 1.016) (layer In1.Cu) (net 4))
+  (via (at 95.758 86.868) (size 0.8) (drill 0.4) (layers F.Cu B.Cu) (net 4) (status 1000000))
+  (segment (start 94.488 76.708) (end 91.694 73.914) (width 1.016) (layer In1.Cu) (net 4) (status 1000000))
+  (segment (start 94.488 85.598) (end 94.488 76.708) (width 1.016) (layer In1.Cu) (net 4) (status 1000000))
+  (segment (start 95.758 86.868) (end 94.488 85.598) (width 1.016) (layer In1.Cu) (net 4) (status 1000000))
+  (segment (start 105.41 107.696) (end 105.41 108.966) (width 0.762) (layer F.Cu) (net 4) (status 1000000))
+  (segment (start 102.616 108.966) (end 102.616 99.314) (width 0.762) (layer F.Cu) (net 4) (status 1000000))
+  (segment (start 100.838 91.948) (end 99.314 90.424) (width 0.762) (layer F.Cu) (net 4) (status 1000000))
+  (segment (start 105.41 108.966) (end 104.902 109.474) (width 0.762) (layer F.Cu) (net 4) (status 1000000))
+  (segment (start 104.902 109.474) (end 103.124 109.474) (width 0.762) (layer F.Cu) (net 4) (status 1000000))
+  (segment (start 99.314 90.424) (end 99.314 87.376) (width 0.762) (layer F.Cu) (net 4) (status 1000000))
+  (segment (start 99.314 87.376) (end 98.806 86.868) (width 0.762) (layer F.Cu) (net 4) (status 1000000))
+  (segment (start 103.124 109.474) (end 102.616 108.966) (width 0.762) (layer F.Cu) (net 4) (status 1000000))
+  (segment (start 102.616 99.314) (end 100.838 97.536) (width 0.762) (layer F.Cu) (net 4) (status 1000000))
+  (segment (start 100.838 97.536) (end 100.838 91.948) (width 0.762) (layer F.Cu) (net 4) (status 1000000))
+  (segment (start 98.806 86.868) (end 95.758 86.868) (width 0.762) (layer F.Cu) (net 4) (status 1000000))
   (segment (start 91.694 73.914) (end 91.694 67.31) (width 1.016) (layer In1.Cu) (net 4))
   (segment (start 91.694 67.31) (end 90.932 66.548) (width 1.016) (layer In1.Cu) (net 4))

Commit message: Add more artwork
Parts:
- removed D3, D4: D_Schottky, Diode_SMD:D_0603_1608Metric
- removed U3: AP1509-33, Package_SO:SO-8_3.9x4.9mm_P1.27mm
- added C10: 22u, Capacitor_SMD:C_1206_3216Metric, F.Cu at (127.8, 105.7)
- added C11: 22u, Capacitor_SMD:C_1206_3216Metric, F.Cu at (106.9, 105.7)
- added C12: 22u, Capacitor_SMD:C_1206_3216Metric, F.Cu at (127.8, 102.7)
- added C13: 10p, Capacitor_SMD:C_0603_1608Metric, F.Cu at (122.6, 105.3)
- added C14: 1u, Capacitor_SMD:C_0603_1608Metric, F.Cu at (117.3, 103.1)
- added C15: 100n, Capacitor_SMD:C_0603_1608Metric, F.Cu at (122.2, 97.4)
- added C16: 10p, Capacitor_SMD:C_0603_1608Metric, F.Cu at (112.1, 105.3)
- added C17: 0.1u, Capacitor_SMD:C_0603_1608Metric, F.Cu at (116.5, 94.3)
- added C18: 0.1u, Capacitor_SMD:C_0603_1608Metric, F.Cu at (118.2, 94.3)
- added F2: CHONK, Fuse:Fuse_1210_3225Metric, F.Cu at (130.8, 92.1)
- added H1: STAR, star-common-lib:star_fancy, F.Cu at (96.5, 95.9)
- added H2: BAC, star-common-lib:bac, F.Cu at (96.4, 102.1)
- added R15: 73.2k, Resistor_SMD:R_0603_1608Metric, F.Cu at (124.4, 105.3)
- added R16: 22.1k, Resistor_SMD:R_0603_1608Metric, F.Cu at (123.4, 102.9)
- added R17: 124k, Resistor_SMD:R_0603_1608Metric, F.Cu at (110.3, 105.3)
- added R18: 22.1k, Resistor_SMD:R_0603_1608Metric, F.Cu at (111.3, 102.9)
- C3, C4: value 100u -> 10u; footprint Capacitor_SMD:C_1210_3225Metric -> Capacitor_SMD:C_0603_1608Metric
- C6: value 100u -> 100n; footprint Capacitor_SMD:C_1210_3225Metric -> Capacitor_SMD:C_0603_1608Metric
- C7: value 100u -> 22u; footprint Capacitor_SMD:C_1210_3225Metric -> Capacitor_SMD:C_1206_3216Metric
- L1: value 47u -> 4.7u; footprint Inductor_SMD:L_Bourns-SRN8040_8x8.15mm -> Inductor_SMD:L_Bourns_SRP5030T
- L2: value 47u -> 2.2u; footprint Inductor_SMD:L_Bourns-SRN8040_8x8.15mm -> Inductor_SMD:L_Bourns_SRP5030T
- U2: value AP1509-50 -> TPS54X94; footprint Package_SO:SO-8_3.9x4.9mm_P1.27mm -> Package_SO:TSSOP-16-1EP_4.4x5mm_P0.65mm
- moved R1 17.0 mm to (108.3, 108.7)
- moved R2 16.2 mm to (126.2, 108.7)
- moved D1 15.8 mm to (105.4, 108.8), turned to 90 degrees
- moved C7 14.7 mm to (106.9, 102.7), turned to 180 degrees
- moved D2 12.0 mm to (129.3, 108.8), turned to 90 degrees
- moved C6 11.4 mm to (112.5, 97.4)
- moved C3 9.57 mm to (114.7, 94.3), turned to 270 degrees
- moved L1 8.14 mm to (107.7, 98.2), turned to 0 degrees
- moved U2 7.75 mm to (117.3, 99.1), turned to 0 degrees
- moved L2 6.81 mm to (127.0, 98.2), turned to 180 degrees
- moved C4 2.42 mm to (120.0, 94.3), turned to 270 degrees
Connections:
- C3 pad 1: +BATT -> GND
- C3 pad 2: GND -> +BATT
- C4 pad 1: +BATT -> GND
- C4 pad 2: GND -> +BATT
- C6 pad 1: +5V -> /SW1
- C6 pad 2: GND -> Net-(C6-Pad2)
- C7 pad 1: +3V3 -> GND
- C7 pad 2: GND -> +5V
- D6 pad 1: +BATT -> Net-(D6-Pad1)
- J4 pad 2: +BATT -> Net-(D6-Pad1)
- L1 pad 1: Net-(D3-Pad1) -> +5V
- L1 pad 2: +5V -> /SW1
- L2 pad 1: Net-(D4-Pad1) -> +3V3
- L2 pad 2: +3V3 -> /SW2
- U2 pad 2: Net-(D3-Pad1) -> Net-(C6-Pad2)
- U2 pad 3: +5V -> /SW1
- U2 pad 5: GND -> +BATT
- U2 pad 6: GND -> Net-(U2-Pad6)
- U2 pad 7: GND -> /FB1
Routing:
- net +5V: track 93.0 -> 68.7 mm, vias 5 -> 4
- net Net-(D3-Pad1): track 14.4 -> 0.00 mm
- net Net-(D4-Pad1): track 14.4 -> 0.00 mm
- net Net-(D6-Pad1): track 0.00 -> 11.3 mm
- net /FB1: track 0.00 -> 7.46 mm
- net /FB2: track 0.00 -> 7.46 mm
- net +BATT: track 92.1 -> 85.9 mm, vias 1 -> 3
- net +3V3: track 102.0 -> 96.1 mm, vias 32 -> 42
- net /SW1: track 0.00 -> 4.67 mm
- net /SW2: track 0.00 -> 4.67 mm
- net Net-(C14-Pad1): track 0.00 -> 3.43 mm
- net Net-(C15-Pad1): track 0.00 -> 2.62 mm
- net Net-(C6-Pad2): track 0.00 -> 2.62 mm
- net GND: track 162.8 -> 160.9 mm, vias 51 -> 41
- net Net-(D2-Pad1): track 2.02 -> 3.10 mm
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- removed copper zone on F.Cu, net GND
Other:
- board text added: "3.3V POWER SUPPLY"
- board text added: "5.0V POWER SUPPLY"

Commit message: Bump rev
Other:
- board text added: "git tag: v1.0.0"
- board text removed: "git tag: v0.0.2"
