File: core/core.sch (KiCad schematic (older format))
At the start: 52 parts, among them J1 Micro_SD_Card, J2 UART_DEBUG, J3 Conn_ARM_JTAG_SWD_10, J4 Conn_01x02, J5 USB_OTG, SW1 SW_Push, SW2 SW_Push, U1 SC18IS600, U2 AP1509-33, U3 AP1509-33

Commit message: Ready CAS for review
Parts:
- C1, C5: DIGIKEY (none) -> 490-13248-1-ND; MANF (none) -> GRM188R6YA106MA73D
- C2, C8: DIGIKEY (none) -> 399-1100-1-ND; MANF (none) -> C0603C104Z3VACTU
- C3, C4, C6, C7: DIGIKEY (none) -> 1276-3364-1-ND; MANF (none) -> CL32A107MPVNNNE
- D1, D2, D5: DIGIKEY (none) -> 475-2816-1-ND; MANF (none) -> LB Q39G-L2OO-35-1
- D3, D4: DIGIKEY (none) -> 478-7798-1-ND; MANF (none) -> SD0603S040S0R2
- F1: DIGIKEY (none) -> MF-FSMF050X-2; MANF (none) -> MF-FSMF050X-2; manf# MF-FSMF050X-2 -> (none)
- J1: DIGIKEY (none) -> 732-3820-1-ND; MANF (none) -> 693072010801; manf# 693072010801 -> (none)
- J2: DIGIKEY (none) -> SAM8981-ND; MANF (none) -> TSM-103-01-L-SV; manf# TSM-103-01-L-SV -> (none)
- J3: DIGIKEY (none) -> SAM13165CT-ND; MANF (none) -> FTSH-105-01-L-DV-K-TR; manf# FTSH-105-01-L-DV-K-TR -> (none)
- J4: DIGIKEY (none) -> WM14505-ND; MANF (none) -> 0026013114
- J5: DIGIKEY (none) -> 900-1051330031TR-ND; MANF (none) -> 1051330031
- L1, L2: DIGIKEY (none) -> SRN8040TA-470MCT-ND; MANF (none) -> SRN8040TA-470M
- R1, R2, R5, R6: DIGIKEY (none) -> 311-1.0KGRCT-ND; MANF (none) -> RC0603JR-071KL
- R10, R11, R12, R7, R8, R9: DIGIKEY (none) -> 311-4.7KGRCT-ND; MANF (none) -> RC0603JR-074K7L
- R3, R4: DIGIKEY (none) -> A130088CT-ND; MANF (none) -> CRGCQ0603J330R
- SW1, SW2: DIGIKEY (none) -> CKN10384CT-ND; MANF (none) -> RS-282G05A3-SM RT
- TP1, TP10, TP11, TP12, TP2, TP3, TP4, TP5, TP6, TP7, TP8, TP9: DIGIKEY (none) -> 36-5014-ND; MANF (none) -> 5014
- U1: DIGIKEY (none) -> 568-13690-1-ND; MANF (none) -> SC18IS600IPW/S8HP
- U2: value AP1509-33 -> AP1509-50; DIGIKEY (none) -> AP1509-50SGDICT-ND; MANF (none) -> AP1509-50SG-13
- U3: DIGIKEY (none) -> AP1509-33SGDICT-ND; MANF (none) -> AP1509-33SG-13

Commit message: fix footprint association
Parts:
- J2: footprint hardware-sch-blocks:TSM-103-01-L-SV -> star-common-lib:TSM-103-01-L-SV
- J3: footprint hardware-sch-blocks:FTSH-105-01-L-DV-K -> star-common-lib:FTSH-105-01-L-DV-K
Changed lines of the file:
@@
 F 0 "J2" H 3758 3181 50  0000 C CNN
 F 1 "UART_DEBUG" H 3758 3090 50  0000 C CNN
-F 2 "hardware-sch-blocks:TSM-103-01-L-SV" H 3650 2900 50  0001 C CNN
+F 2 "star-common-lib:TSM-103-01-L-SV" H 3650 2900 50  0001 C CNN
 F 3 "~" H 3650 2900 50  0001 C CNN
 F 4 "" H 3650 2900 50  0001 C CNN "manf#"
@@
 F 0 "J3" H 3800 2100 50  0000 R CNN
 F 1 "Conn_ARM_JTAG_SWD_10" V 3650 2000 50  0000 R CNN
-F 2 "hardware-sch-blocks:FTSH-105-01-L-DV-K" H 4100 1550 50  0001 C CNN
+F 2 "star-common-lib:FTSH-105-01-L-DV-K" H 4100 1550 50  0001 C CNN
 F 3 "http://infocenter.arm.com/help/topic/com.arm.doc.ddi0314h/DDI0314H_coresight_components_trm.pdf" V 3750 300 50  0001 C CNN
 F 4 "" H 4100 1550 50  0001 C CNN "manf#"

Commit message: fix usb connector
Parts:
- J5: footprint Connector_USB:USB_Micro-B_Molex-105133-0001 -> Connector_USB:USB_Micro-B_Molex-105017-0001; DIGIKEY 900-1051330031TR-ND -> WM1399CT-ND; MANF 1051330031 -> 1050170001
Changed lines of the file:
@@
 F 0 "J5" H 7357 1567 50  0000 C CNN
 F 1 "USB_OTG" H 7357 1476 50  0000 C CNN
-F 2 "Connector_USB:USB_Micro-B_Molex-105133-0001" H 7450 1050 50  0001 C CNN
+F 2 "Connector_USB:USB_Micro-B_Molex-105017-0001" H 7450 1050 50  0001 C CNN
 F 3 " ~" H 7450 1050 50  0001 C CNN
-F 4 "900-1051330031TR-ND" H 7300 1100 50  0001 C CNN "DIGIKEY"
-F 5 "1051330031" H 7300 1100 50  0001 C CNN "MANF"
+F 4 "WM1399CT-ND" H 7300 1100 50  0001 C CNN "DIGIKEY"
+F 5 "1050170001" H 7300 1100 50  0001 C CNN "MANF"
 	1    7300 1100
 	1    0    0    -1

Commit message: Update block schematics and layout
Connections:
- net INT_IMU: no longer names the net of U1.1 (GPIO0)
- no-connect marks 15 -> 16
Changed lines of the file:
@@
 Wire Wire Line
 	9150 4550 8900 4550
-NoConn ~ 8900 5000
 Wire Wire Line
 	9150 3650 8900 3650
@@
 Text Notes 7650 1800 0    50   ~ 0
 USB
-Text Label 7750 2750 2    50   ~ 0
-SPI2_nSS2
-Wire Wire Line
-	8000 2750 7750 2750
 NoConn ~ 1350 7000
 NoConn ~ 4400 6950
@@
 $EndComp
 Wire Wire Line
-	1250 5350 1150 5350
-Text Label 1150 5350 2    50   ~ 0
-INT_IMU
-Wire Wire Line
 	650  5650 1250 5650
 Wire Wire Line
@@
 F5 "SCL" I R 9350 1400 50
 $EndSheet
+NoConn ~ 1250 5350
+Text Label 9150 5000 0    50   ~ 0
+SPI3_nSS2
+Wire Wire Line
+	9150 5000 8900 5000
+NoConn ~ 8000 2750
 $EndSCHEMATC

Commit message: Address comments
Connections:
- net +BATT: now also J4.1 (Pin_1); no longer J4.2 (Pin_2)
- net GND: now also J4.2 (Pin_2); no longer J4.1 (Pin_1)
Other:
- note added: "CAS Core Module Schematic"
- moved on the sheet: J4
Changed lines of the file:
@@
-$EndComp
-$Comp
-L Connector_Generic:Conn_01x02 J4
-U 1 1 5F0BA043
-P 6100 3150
-F 0 "J4" H 6018 2825 50  0000 C CNN
-F 1 "Conn_01x02" H 6018 2916 50  0000 C CNN
-F 2 "star-common-lib:Molex_Mini-Fit_Jr_5569-02A2_2x01_P4.20mm_Horizontal" H 6100 3150 50  0001 C CNN
-F 3 "~" H 6100 3150 50  0001 C CNN
-F 4 "WM14505-ND" H 6100 3150 50  0001 C CNN "DIGIKEY"
-F 5 "0026013114" H 6100 3150 50  0001 C CNN "MANF"
-	1    6100 3150
-	-1   0    0    1
 $EndComp
 $Comp
 L power:+BATT #PWR034
 U 1 1 5F0C02D9
-P 6550 3050
-F 0 "#PWR034" H 6550 2900 50  0001 C CNN
-F 1 "+BATT" H 6565 3223 50  0000 C CNN
-F 2 "" H 6550 3050 50  0001 C CNN
-F 3 "" H 6550 3050 50  0001 C CNN
-	1    6550 3050
+P 6150 3000
+F 0 "#PWR034" H 6150 2850 50  0001 C CNN
+F 1 "+BATT" H 6165 3173 50  0000 C CNN
+F 2 "" H 6150 3000 50  0001 C CNN
+F 3 "" H 6150 3000 50  0001 C CNN
+	1    6150 3000
 	1    0    0    -1
 $EndComp
@@
 L power:GND #PWR035
 U 1 1 5F0C070B
-P 6550 3150
-F 0 "#PWR035" H 6550 2900 50  0001 C CNN
-F 1 "GND" H 6555 2977 50  0000 C CNN
-F 2 "" H 6550 3150 50  0001 C CNN
-F 3 "" H 6550 3150 50  0001 C CNN
-	1    6550 3150
-	1    0    0    -1
-$EndComp
-Wire Wire Line
-	6300 3050 6550 3050
-Wire Wire Line
-	6550 3150 6300 3150
+P 6150 3100
+F 0 "#PWR035" H 6150 2850 50  0001 C CNN
+F 1 "GND" H 6155 2927 50  0000 C CNN
+F 2 "" H 6150 3100 50  0001 C CNN
+F 3 "" H 6150 3100 50  0001 C CNN
+	1    6150 3100
+	1    0    0    -1
+$EndComp
+Wire Wire Line
+	6400 3100 6150 3100
+Wire Wire Line
+	6150 3000 6400 3000
 Text Notes 6150 3450 0    50   ~ 0
 Battery Connector
@@
 I2C3_SDA
 Text Label 1100 7300 2    50   ~ 0
-I2C3_SDA
+I2C3_SCL
 Wire Notes Line
 	6950 1900 11150 1900
@@
 	9150 5000 8900 5000
 NoConn ~ 8000 2750
+$Comp
+L Connector_Generic:Conn_01x02 J4
+U 1 1 5F0BA043
+P 6600 3000
+F 0 "J4" H 6518 2675 50  0000 C CNN
+F 1 "Conn_01x02" H 6518 2766 50  0000 C CNN
+F 2 "star-common-lib:Molex_Mini-Fit_Jr_5569-02A2_2x01_P4.20mm_Horizontal" H 6600 3000 50  0001 C CNN
+F 3 "~" H 6600 3000 50  0001 C CNN
+F 4 "WM14505-ND" H 6600 3000 50  0001 C CNN "DIGIKEY"
+F 5 "0026013114" H 6600 3000 50  0001 C CNN "MANF"
+	1    6600 3000
+	1    0    0    -1
+$EndComp
+Text Notes 7350 7500 0    50   ~ 0
+CAS Core Module Schematic
 $EndSCHEMATC
