File: core/core.sch (KiCad schematic (older format))
At the start: 63 parts, among them J1 Micro_SD_Card, J2 UART_DEBUG, J3 Conn_ARM_JTAG_SWD_10, J4 Conn_01x02, J5 USB_OTG, SW1 RESET, SW2 USER, U1 SC18IS600, U2 TPS54X94, U4 USBLC6-2SC6

Commit message: Add more artwork
Parts:
- added F2: CHONK, Fuse:Fuse_1210_3225Metric, symbol Device:Polyfuse_Small
- added H1: STAR, star-common-lib:star_fancy, symbol Mechanical:MountingHole
- added H2: BAC, star-common-lib:bac, symbol Mechanical:MountingHole
- C13, C14, C15, C16, C6: footprint Capacitor_SMD:C_1206_3216Metric -> Capacitor_SMD:C_0603_1608Metric
- F1: DIGIKEY MF-FSMF050X-2 -> MF-FSMF050X-2CT-ND
- L2: value 2.2 -> 2.2u
- R15: value 73.2 -> 73.2k; DIGIKEY 311-2950-1-ND -> P73.2KDBCT-ND; MANF RT1206DRD0773R2L -> ERA-3AEB7322V
- R16, R18: value 22.1 -> 22.1k; DIGIKEY A110384CT-ND -> P22.1KDBCT-ND; MANF 6-1625868-0 -> ERA-3AEB2212V
- R17: value 124 -> 124k; DIGIKEY P124DBCT-ND -> P124KDBCT-ND; MANF ERA-3AEB1240V -> ERA-3AEB1243V
Connections:
- net +BATT: now also F2.1; no longer D6.1 (K), J4.2 (Pin_2)
- net FB1: now also C16.2, R17.2, R18.1; no longer C13.2, R15.2, R16.1
- net FB2: now also C13.2, R15.2, R16.1; no longer C16.2, R17.2, R18.1
- net GND: now also U2.4 (PGND1)
- net SW1: now also L1.2; no longer L2.2
- net SW2: now also L2.2; no longer L1.2
- new net: D6.1 (K), F2.2, J4.2 (Pin_2)
Other:
- note removed: "CAS Core Module Schematic"
